File: 440MHz.kicad_sch (KiCad schematic)
At the start: 48 parts, among them J5 BWSMA-KWE-Z001, U10 74LVC1GU04DRL, U7 GRF5604, U9 SKYA21003

Commit message: Reduce hole sizes and add more holes on PA
Meet spec requirements.

Signed-off-by: Corey Minyard <corey@minyard.net>
Parts:
- C38, C51: value 5.1pF -> 5.1pF 1%
- C50: value 15pF -> 15pF 1%
- C52, C68: value 2.2pF -> 2.2pF 1%
- C54: value 12pF -> 12pF 1%
- C57: value 10pF -> 10pF 1%
- C58, C61: value 33pF -> 33pF 1%
- C62: value 2pF -> 2pF 1%
- C64: value 28pF -> 28pF 1%
- C66: value 1.8pF -> 1.8pF 1%
- L10: value 43nH -> 43nH 2%
- L11, L17: value 27nH -> 27nH 2%
- L12: value 22nH -> 22nH 2%
- L13: value 10nH -> 10nH 2%
- L15: value 2.2nH -> 2.2nH 2%
- L19: value 15nH -> 15nH 2%
Changed lines of the file:
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@@
 			)
 		)
-		(property "Value" "5.1pF"
+		(property "Value" "5.1pF 1%"
 			(at 85.344 150.876 90)
 			(effects
@@
 			)
 		)
-		(property "Value" "43nH"
+		(property "Value" "43nH 2%"
 			(at 68.834 80.772 90)
 			(effects
@@
 			)
 		)
-		(property "Value" "28pF"
-			(at 249.936 84.328 90)
+		(property "Value" "28pF 1%"
+			(at 249.936 82.296 90)
 			(effects
 				(font
@@
 			)
 		)
-		(property "Value" "33pF"
+		(property "Value" "33pF 1%"
 			(at 227.076 84.328 90)
 			(effects
@@
 			)
 		)
-		(property "Value" "10nH"
+		(property "Value" "10nH 2%"
 			(at 129.032 87.376 90)
 			(effects
@@
 			)
 		)
-		(property "Value" "15pF"
+		(property "Value" "15pF 1%"
 			(at 61.976 83.566 90)
 			(effects
@@
 			)
 		)
-		(property "Value" "27nH"
+		(property "Value" "27nH 2%"
 			(at 64.262 157.226 90)
 			(effects
@@
 			)
 		)
-		(property "Value" "15nH"
+		(property "Value" "15nH 2%"
 			(at 47.244 80.772 90)
 			(effects
@@
 			)
 		)
-		(property "Value" "12pF"
+		(property "Value" "12pF 1%"
 			(at 96.266 84.328 90)
 			(effects
@@
 			)
 		)
-		(property "Value" "1.8pF"
+		(property "Value" "1.8pF 1%"
 			(at 260.096 84.328 90)
 			(effects
@@
 			)
 		)
-		(property "Value" "2.2pF"
-			(at 49.784 73.406 90)
+		(property "Value" "2.2pF 1%"
+			(at 51.816 73.406 90)
 			(effects
 				(font
@@
 			)
 		)
-		(property "Value" "2.2pF"
-			(at 79.756 84.328 90)
+		(property "Value" "2.2pF 1%"
+			(at 79.502 81.788 90)
 			(effects
 				(font
@@
 			)
 		)
-		(property "Value" "10pF"
+		(property "Value" "10pF 1%"
 			(at 120.904 82.296 90)
 			(effects
@@
 			)
 		)
-		(property "Value" "27nH"
+		(property "Value" "27nH 2%"
 			(at 82.804 130.302 90)
 			(effects
@@
 			)
 		)
-		(property "Value" "5.1pF"
+		(property "Value" "5.1pF 1%"
 			(at 75.946 154.686 90)
 			(effects
@@
 			)
 		)
-		(property "Value" "2pF"
-			(at 237.236 84.328 90)
+		(property "Value" "2pF 1%"
+			(at 237.236 83.058 90)
 			(effects
 				(font
@@
 			)
 		)
-		(property "Value" "22nH"
+		(property "Value" "22nH 2%"
 			(at 85.344 80.772 90)
 			(effects
@@
 			)
 		)
-		(property "Value" "33pF"
+		(property "Value" "33pF 1%"
 			(at 138.684 82.296 90)
 			(effects
@@
 			)
 		)
-		(property "Value" "2.2nH"
+		(property "Value" "2.2nH 2%"
 			(at 239.014 80.772 90)
 			(effects
