File: radio2.kicad_sch (KiCad schematic)
At the start: 27 parts, among them Y1 OW2EL89CENUXK7YLC-40M

Commit message: More re-layout for the new design
Signed-off-by: Corey Minyard <corey@minyard.net>
Parts:
- removed R43, R44: 0Ω, Resistor_SMD:R_0402_1005Metric, symbol Device:R
- removed U?: CC1125RHBR, footprints:RHB32_3P45X3P45_TEX, symbol Local ICs:CC1125RHBR
- added U14: CC1125RHBR, footprints:RHB32_3P45X3P45_TEX, symbol Local ICs:CC1125RHBR
Connections:
- net +5V is gone; now on net +3.3V: C53.2, R16.2
- net +3.3V: now also U14.1 (VDD_GUARD), U14.12 (DVDD), U14.13 (AVDD_IF), U14.15 (AVDD_RF), U14.22 (AVDD_SYNTH1), U14.25 (AVDD_PFD_CHP), U14.27 (AVDD_SYNTH2), U14.28 (AVDD_XOSC), U14.5 (DVDD)
- net 440_RX_N: now also U14.20 (LNA_N)
- net 440_RX_P: now also U14.19 (LNA_P)
- net 440_TRX_SW: now also U14.18 (TRX_SW)
- net GND: now also U14.30 (XOSC_Q1), U14.33 (EPAD)
- net RADIO2_RESET_N: now also U14.2 (RESET_N)
- net RADIO2_SPI_SSEL: now also U14.11 (CSN)
- net at C49.1, L18.1: now also U14.17 (PA)
- net at C28.2: now also U14.6 (DCPL)
- net at C14.2: now also U14.21 (DCPL_VCO)
- net at R7.2: now also U14.14 (RBIAS)
- net at C16.1: now also U14.23 (LPF0)
- net at C16.2: now also U14.24 (LPF1)
- net at C18.2: now also U14.26 (DCPL_PFD_CHP)
- net at C17.2: now also U14.29 (DCPL_XOSC)
- net at C29.1: now also U14.32 (EXT_XOSC)
- new net RADIO2_GPIO0: U14.10 (GPIO0)
- new net RADIO2_GPIO2: U14.4 (GPIO2)
- new net RADIO2_GPIO3: U14.3 (GPIO3)
- new net RADIO_SPI_MISO: U14.9 (SO(GPIO1))
- new net RADIO_SPI_MOSI: U14.7 (SI)
- new net RADIO_SPI_SCLK: U14.8 (SCLK)
- no-connect marks 4 -> 2
